File: _pcb/Harp Motor device H2-module v1.0/Harp Motor device H2-module v1.0.sch (EAGLE design)
At the start: 45 parts, among them IC1 FT232RL, IC3 LP5907MFX-3.3, IC7 USBLC6-2SC6, IC8 ATXMEGA32A4U, X15 Main_plug, X3 USB_MINI_B

Commit message: Harp Motor device H2 - design
still first steps on Eagle Harp Motor device H2 design
Parts:
- removed LICK_0, LICK_1: 1x3 case, con-molex:22-23-2031
- removed REWARD_VALVES: 1x4 case, con-molex:22-23-2041
- added J1, J2: BNCPTH, SparkFun-Connectors:BNCPTH
- added J3: POWER_JACK, SparkFun-Connectors:POWER_JACK
- added X1, X2: 22-23-2051, con-molex:22-23-2051
- added X4, X7: 1x4 case, con-molex:22-23-2041
- added X5: 1x3 case, con-molex:22-23-2031
- added X6: CLCK_JACK, harp input expander:STEREO_JACK
- added X8: 22-23-2021, con-molex:22-23-2021
Connections:
- removed net HARP_H1_BOARD_RX: X15.3
- removed net HARP_H1_BOARD_TX: X15.2
- new net HARP_H1_RX: X1-3.S
- new net HARP_H1_TX: X1-4.S
- new net N$4: X1-5.S, X2-5.S, X4-4.S
- net +3V3: now also X5-3.S; no longer LICK_0-3.S, LICK_1-3.S
- net GND: now also X1-1.S, X2-1.S, X4-1.S, X5-1.S, X6.5; no longer LICK_0-1.S, LICK_1-1.S
- net HARP_H1_CLOCK_IN: now also X1-2.S; no longer X15.4
Other:
- note added: "5V~24V inputs (??)"
- note added: "CHECK VOLTAGE LEVEL OUTPUT!!!"
- note added: "InOut H1 Harp interface"
- note added: "in Clock input"
- note added: "in Emergency Button"
- note added: "in Hall Effect sensor"
- note added: "in jumpers to setup/test open or closed loop control??"
- note added: "in rotary encoder"
- note added: "in sphere rotation signal"
- note added: "in stage rotation signal ?? 2 signals??"
- note added: "level translatioon 5V -> 3V3"
- note added: "level translatioon 5V~24V -> 3V3"
- note added: "out step motor driver"
- note added: "to u; PullDown"
- note removed: "-to review USBDP & USBDP pin switched!!!"
- note removed: "-to review pinout upside-down!!!"
- moved on the sheet: TP4, TP5, TP6, TP8, TP9
