File: _pcb/Harp Motor device H2-module v1.0/Harp Motor H2-module v1.0.sch (EAGLE design)
At the start: 84 parts, among them IC1 FT232RL, IC10 OPA365, IC11 74LVC1G125DBV, IC12 74LVC1G125DBV, IC2 74LVC1G125DBV, IC3 LP5907MFX-3.3, IC7 USBLC6-2SC6, IC8 ATXMEGA32A4U, IC9 TLV70033DDCR, T1 DMG1012UW??, T2 DMG1012UW??, T3 DMG1012UW??, X1 be sure about plug type, X2 Rot_Encoder, X3 EMRG_BUTT_IN_NO, X4 Hall_Effect, X5 STEP_MOTOR, X6 USB_MINI_B, X7 DC_JACK2.1MM

Commit message: Harp Motor device H2-module v1.0 - BOM not finished
Harp Motor device H2-module v1.0
- BOM committed; not yet finished
Parts:
- removed CLKIN: CLCK_JACK, harp input expander:STEREO_JACK
- added X8: CLCK_JACK, Harp Motor H2-module v1.0:STEREO_JACK
- C1, C12, C14, C16, C17, C18, C25, C26, C27, C28, C29, C3, C5, C7, C9: DIGIKEY_PN 445-5932-1-ND -> (none); NOTES - -> (none); TYPE SMD -> (none)
- C10, C11: NOTES - -> (none); TYPE SMD -> (none)
- C15: value 4.7uF DNI -> 4.7uF; NOTES - -> (none); TYPE SMD -> (none)
- C23, C24: device rcl:C-EUC0603 -> Harp Motor H2-module v1.0:C-EUC0603K; NOTES - -> (none); OEPS (none) -> OEPS010018; TYPE SMD -> (none)
- C41, C42: device rcl:C-EUC0402 -> Harp Motor H2-module v1.0:C-EUC0402K; MPN (none) -> TBD; OEPS (none) -> TBD
- C8: device Harp Motor H2-module v1.0:C-EUC0603 -> Harp Motor H2-module v1.0:C-EUC0603K
- IC1: device VestibularVR H1-module v1.0:FT232RL -> Harp Motor H2-module v1.0:FT232RL
- IC10: device CNP-ics 2:OPA365 -> Harp Motor H2-module v1.0:OPA365; MPN (none) -> OEPS080019=TLV272CDGKR; OEPS (none) -> TBD
- IC11, IC12, IC2: MPN (none) -> SN74LVC1G125DBVT; OEPS (none) -> OEPS080029
- IC3: device VestibularVR H1-module v1.0:TLV700XX -> Harp Motor H2-module v1.0:TLV700XX; NOTES - -> (none); TYPE SMD -> (none)
- IC7: device VestibularVR H1-module v1.0:USBLC6-2SC6 -> Harp Motor H2-module v1.0:USBLC6-2SC6
- IC8: device VestibularVR H1-module v1.0:XMEGA-A4_AT-XMEGA-XXA4-AUTQFP44 -> Harp Motor H2-module v1.0:XMEGA-A4_AT-XMEGA-XXA4-AUTQFP44; MPN (none) -> ATXMEGA32A4U-AUR
- IC9: value TLV70033DDCR -> LP5907MFX-3.3; device harp input expander:TLV700XX -> Harp Motor H2-module v1.0:TLV700XX; MPN TLV70033DDCR -> LP5907MFX-3.3/NOPB; NOTES - -> (none); OEPS (none) -> OEPS080016; TYPE SMD -> (none)
- OSC1: device VestibularVR H1-module v1.0:OSCILLATOR -> Harp Motor H2-module v1.0:OSCILLATOR
- R1, R12, R18, R2, R34, R6, R8: DIGIKEY_PN 541-10.0KLDKR-ND -> (none)
- R10: value DNI -> DNI 0R; DIGIKEY_PN - -> (none); MPN DNI -> RC0402JR-070RL; OEPS DNI -> OEPS020001
- R11: DIGIKEY_PN a de 0R -> (none); MPN a de 0R -> RC0402JR-070RL; OEPS a de 0R -> OEPS020001
- R13: value DNI -> 10k; DIGIKEY_PN - -> (none); MPN - -> CRCW040210K0FKED; OEPS - -> OEPS020030
- R14, R15, R16: DIGIKEY_PN - -> (none)
- R17, R19: value 10k 1% -> 10k; device rcl:R-EU_R0402 -> Harp Motor H2-module v1.0:R-US_R0402; MPN (none) -> CRCW040210K0FKED; OEPS (none) -> OEPS020030
- R20: device rcl:R-EU_R0402 -> Harp Motor H2-module v1.0:R-EU_R0402; MPN (none) -> TBD; OEPS (none) -> TBD
- R21: device rcl:R-EU_R0402 -> Harp Motor H2-module v1.0:R-EU_R0402; MPN (none) -> ERJ-2RKF1502X; OEPS (none) -> OEPS020015
- R3: DIGIKEY_PN 541-1.00MLCT-ND -> (none)
- R4: value 0R DNI -> div tensao ADC; DIGIKEY_PN ?? -> (none); MPN TBD ? -> n.a
- R5: DIGIKEY_PN qwee -> (none); MPN as -> ERJ-PA2J100X; OEPS xx -> OEPS020041
- R7: value 10k DNI -> div tensao ADC; DIGIKEY_PN 541-10.0KLDKR-ND -> (none); MPN CRCW040210K0FKED -> n.a.; OEPS OEPS020030 -> TBD
- R9: value 100R DNI -> DNI 100R; DIGIKEY_PN para 100R -> (none); MPN para 100R -> ERJ-2RKF1000X; OEPS OEPS para100R -> OEPS020004
- T1, T2, T3: value DMG1012UW?? -> DMG1012UW; device VestibularVR H1-module v1.0:DMG1012UW-7 -> Harp Motor H2-module v1.0:DMG1012UW-7; OEPS ?? escolhido muito power?? -> OEPS060010
- X1: value be sure about plug type -> 1x5 MAIN PLUG
- X2: value Rot_Encoder -> 1x5 case; MPN (none) -> 282834-5; OEPS (none) -> TBD
- X3: value EMRG_BUTT_IN_NO -> 1x2 case; MPN (none) -> 282834-2; OEPS (none) -> TBD
- X4: value Hall_Effect -> 1x3 case; MF - -> (none)
- X5: value STEP_MOTOR -> 1x5 case; MPN (none) -> 282834-5; OEPS (none) -> TBD
- X6: device VestibularVR H1-module v1.0:USB_MINI_B -> Harp Motor H2-module v1.0:USB_MINI_B
- X7: device harp camera controller:DC_JACK2.1MM -> Harp Motor H2-module v1.0:DC_JACK2.1MM; DIGIKEY_PN DIGIKEY N.A. -> (none); MOUSER_PN 163-179PH -> (none); NOTES - -> (none); OEPS (none) -> OEPS070026; TYPE TH -> (none)
Connections:
- net +3V3_U renamed V+
- net GND: now also X8.5; no longer CLKIN.5
- net N$103: now also X8.1; no longer CLKIN.1
- net U_CLOCK_IN: now also X8.4; no longer CLKIN.4
