File: Hardware/PCB/VestibularH2.sch (EAGLE design)
At the start: 84 parts, among them IC1 FT232RL, IC10 THS4281DBVT, IC11 SN74LVC1G125DBVT, IC12 SN74LVC1G125DBVT, IC2 SN74LVC1G125DBVT, IC3 LP5907MFX-3.3, IC7 USBLC6-2SC6, IC8 ATXMEGA32A4U, IC9 LP5907MFX-3.3, T1 DMG1012UW, T2 DMG1012UW, T3 DMG1012UW, X1 1x5 MAIN PLUG, X2 1x5 case, X3 1x2 case, X4 1x3 case, X5 1x5 case, X6 USB_MINI_B, X7 DC_JACK2.1MM, X8 CLCK_JACK

Commit message: Replaced files with PCB version 1.1.
Parts:
- removed R10: DNI 0R, Harp Motor H2-module v1.0:R-US_R0402
- removed R11: 0R, Harp Motor H2-module v1.0:R-US_R0402
- removed R14, R15, R16: DNI, Harp Motor H2-module v1.0:R-US_R0402
- removed T1, T2, T3: DMG1012UW, Harp Motor H2-module v1.0:DMG1012UW-7
- added IC4, IC5, IC6: M74VHC1GT126DT1G, Harp Motor H2-module v1.0:M74VHC1GT126DT1G
- C15: value DNI 4.7uF -> DNI; MPN C1608X6S1C475K080AC -> DNI; OEPS OEPS010018 -> DNI
- IC11, IC12, IC2: value SN74LVC1G125DBVT -> M74VHC1GT126DT1G; device Harp Motor H2-module v1.0:74LVC1G125DBV -> Harp Motor H2-module v1.0:M74VHC1GT126DT1G; DIGIKEY_PN (none) -> M74VHC1GT126DT1GOSDKR-ND; MPN SN74LVC1G125DBVT -> M74VHC1GT126DT1G; OEPS OEPS080029 -> OEPS080017
- R9: value DNI 100R -> DNI; MPN ERJ-2RKF1000X -> DNI; OEPS OEPS020004 -> DNI
Connections:
- removed net N$51: R10.1, R11.1, X4-2.S
- net +3V3: now also IC11.OE, IC12.OE, IC2.OE; no longer R11.2
- net +5V: now also IC4.OE, IC4.VCC, IC5.OE, IC5.VCC, IC6.OE, IC6.VCC, X4-2.S; no longer R10.2, R14.2, R15.2, R16.2
- net ENCODER_A_PHASE: now also IC11.A; no longer IC12.I
- net ENCODER_B_PHASE: now also IC2.A; no longer IC11.I
- net GND: now also IC4.GND, IC5.GND, IC6.GND; no longer IC11.OE, IC12.OE, IC2.OE, T1.S, T2.S, T3.S
- net HARP_H2_CLOCK_OUT: now also IC12.Y; no longer IC2.O
- net HARP_H2_RX: now also X1.2; no longer X1.3
- net HARP_H2_TX: now also X1.3; no longer X1.2
- net STEP_DIRECTION: now also IC5.Y; no longer R15.1, T1.D
- net STEP_ENABLE: now also IC6.Y; no longer R14.1, T3.D
- net STEP_PULSE: now also IC4.Y; no longer R16.1, T2.D
- net U_CLOCK_IN: now also IC12.A; no longer IC2.I
- net U_ENCODER_A_PHASE: now also IC11.Y; no longer IC12.O
- net U_ENCODER_B_PHASE: now also IC2.Y; no longer IC11.O
- net U_STEP_DIRECTION: now also IC5.A, R13.2; no longer R12.2, T1.G
- net U_STEP_ENABLE: now also IC6.A, IC8.PC3/OC0D/TXD0, R6.2; no longer IC8.PC0/OC0A/SDA, R13.2, T3.G
- net U_STEP_PULSE: now also IC4.A, IC8.PC0/OC0A/SDA, R12.2; no longer IC8.PC3/OC0D/TXD0, R6.2, T2.G
Other:
- note removed: "power rail: - Vcc to stepper drive controller optos - DM542 stepper drive controller Vcc: = 5V~24V >> output voltage here can be 5V - Imax = ???"
- moved on the sheet: C10, C11, C12, C13, C14, C15, C17, C18, IC3, R1, R12, R13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

Commit message: Created the schematic with new ios.
Parts:
- added C19, C20, C21, C22, C30, C31: 100nF, Harp Motor H2-module v1.0:C-EUC0402K
- added IC13, IC14, IC15, IC16, IC17, IC18: M74VHC1GT126DT1G, Harp Motor H2-module v1.0:M74VHC1GT126DT1G
- added R10, R11, R14: 10k, Harp Motor H2-module v1.0:R-US_R0402
- added X10: 1x3 case, Harp Motor H2-module v1.0:22-23-2031
- added X9: 1x5 case, Harp Motor H2-module v1.0:22-23-2051
Connections:
- net ENCODER_A_PHASE renamed INPUT1
- net ENCODER_B_PHASE renamed INPUT0
- net U_ENCODER_A_PHASE renamed U_PH_B
- net U_ENCODER_B_PHASE renamed U_PH_A
- new net BRAKE: IC17.Y, X10-3.S
- new net ENDSTOP: IC18.A, X10-2.S
- new net IN0: IC13.A, X9-2.S
- new net IN1: IC14.A, X9-3.S
- new net OUTPUT0: IC16.Y, X9-4.S
- new net OUTPUT1: IC15.Y, X9-5.S
- new net UC_BRAKE: IC17.A, R14.2
- new net UC_ENDSTOP: IC18.Y, IC8.PC7/SCK/TXD1/CLKO/EVO
- new net UC_INPUT0: IC13.Y, IC8.OCB1/XCK1/MOSI/PD5
- new net UC_INPUT1: IC14.Y, IC8.D-/RXD1/MISO/PD6
- new net UC_OUTPUT0: IC16.A, R10.2
- new net UC_OUTPUT1: IC15.A, R11.2
- net +3V3: now also C19.1, C20.1, C21.1, IC13.OE, IC13.VCC, IC14.OE, IC14.VCC, IC18.OE, IC18.VCC
- net +5V: now also C22.1, C30.1, C31.1, IC15.OE, IC15.VCC, IC16.OE, IC16.VCC, IC17.OE, IC17.VCC
- net GND: now also C19.2, C20.2, C21.2, C22.2, C30.2, C31.2, IC13.GND, IC14.GND, IC15.GND, IC16.GND, IC17.GND, IC18.GND, R10.1, R11.1, R14.1, X10-1.S, X9-1.S
Other:
- note added: "extra digital ios"
- note added: "extra motor control"
- note added: "ligar no uc onde der jeito"

Commit message: Finalized the layout.
Co-Authored-By: David Palma <78764277+davidpalma666@users.noreply.github.com>
Connections:
- net UC_BRAKE: now also IC8.PB3/ADC11/DAC1
- net UC_OUTPUT0: now also IC8.PB1/ADC9
- net UC_OUTPUT1: now also IC8.PA7/ADC7/AC0-OUT
Other:
- note removed: "ligar no uc onde der jeito"
- moved on the sheet: C19, C20, C21, C22, C30, C31, IC13, IC14, IC15, IC16, IC17, IC18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
